File: labs/lab1/lab1.kicad_sch (KiCad schematic)
At the start: 0 parts

Commit message: added lab1
Parts:
- added C1: 0.1u, Capacitor_SMD:C_0603_1608Metric, symbol Device:C
- added H1, H2, H3: MountingHole, MountingHole:ToolingHole_1.152mm, symbol Mechanical:MountingHole
- added H4, H5, H6, H7: MountingHole, MountingHole:MountingHole_3.2mm_M3_DIN965, symbol Mechanical:MountingHole
- added U1: ADS1114IDGS, Package_SO:TSSOP-10_3x3mm_P0.5mm, symbol Analog_ADC:ADS1114IDGS
- added V1: 0, symbol Simulation_SPICE:VDC
- added V2, V3, V4, V5, V6, V7, V8: 3.3, symbol Simulation_SPICE:VDC
Connections:
- new net +3V3A: C1.1, U1.8 (VDD)
- new net ADC_IN: U1.2 (ALERT/RDY)
- new net GND: V1.2, V2.2, V3.2, V4.2, V5.2, V6.2, V7.2, V8.2
- new net GNDA: C1.2, U1.1 (ADDR), U1.3 (GND), U1.5 (AIN1)
- new net I2C_SCL: U1.10 (SCL)
- new net I2C_SDA: U1.9 (SDA)
- new net OUT: U1.4 (AIN0)
- new net relay_0: V1.1
- new net relay_1: V2.1
- new net relay_2: V3.1
- new net relay_3: V4.1
- new net relay_4: V5.1
- new net relay_5: V6.1
- new net relay_6: V7.1
- new net relay_7: V8.1
Other:
- added sheet FEE_1 (modules/FEE.kicad_sch)
- added sheet FEE_2 (modules/FEE.kicad_sch)
- added sheet FEE_3 (modules/FEE.kicad_sch)
- added sheet FEE_4 (modules/FEE.kicad_sch)
- added sheet FEE_5 (modules/FEE.kicad_sch)
- added sheet FEE_6 (modules/FEE.kicad_sch)
- added sheet FEE_7 (modules/FEE.kicad_sch)
- added sheet FEE_8 (modules/FEE.kicad_sch)
- added sheet micro_controller (modules/controller.kicad_sch)
- added sheet power (modules/power.kicad_sch)
- note added: ".OPTIONS reltol=0.01 abstol=1e-9 vntol=0.01"
- note added: "GNDA - detector ground to be referenced at hearth GND - digital groud to be kept floating"
