File: labs/lab2/gtr.kicad_sch (KiCad schematic)
At the start: 1 part, among them U1 XC7A35T-FGG484

Commit message: work on lection 1
Parts:
- U1: footprint (none) -> Package_BGA:BGA484C100P22X22_2300X2300X260
Changed lines of the file:
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@@
 			)
 		)
-		(property "Footprint" ""
+		(property "Footprint" "Package_BGA:BGA484C100P22X22_2300X2300X260"
 			(at 99.06 154.94 0)
 			(effects
@@
 			)
 		)
-		(property "Footprint" ""
+		(property "Footprint" "Package_BGA:BGA484C100P22X22_2300X2300X260"
 			(at 99.06 86.36 0)
 			(effects
