File: labs/lab2/lab2.kicad_sch (KiCad schematic)
At the start: 1 part, among them U1 XC7A35T-FGG484

Commit message: work on lection 1
Parts:
- U1: footprint (none) -> Package_BGA:BGA484C100P22X22_2300X2300X260
Connections:
- net GND: now reaches U1.A11 (GND)
- net GND: now also U1.A12 (GND), U1.A2 (GND), U1.A22 (GND), U1.A3 (GND), U1.A5 (GND), U1.A7 (GND), U1.A9 (GND), U1.AA12 (GND), U1.AA2 (GND), U1.AA22 (GND), U1.AB19 (GND), U1.AB9 (GND)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
